File: PCB Test/PCB Test.kicad_sch (KiCad schematic)
At the start: 50 parts, among them J1 Conn_02x02_Counter_Clockwise, J2 Conn_02x05_Odd_Even, J3 Conn_02x02_Odd_Even, J4 Conn_02x02_Odd_Even, J5 Conn_02x02_Odd_Even, J6 Conn_02x03_Odd_Even, Q2 NMOS, Q3 NMOS, SW1 SW_Push, SW2 SW_Push, SW3 SW_Push, U1 ATmega4808-A, U5 MCP1700x-330xxTO

Commit message: Light polishing
Parts:
- J2: footprint Connector_PinHeader_1.00mm:PinHeader_2x05_P1.00mm_Vertical_SMD -> Connector_PinHeader_1.00mm:PinHeader_2x06_P1.00mm_Vertical
- J6: footprint Connector_PinSocket_1.00mm:PinSocket_2x03_P1.00mm_Vertical_SMD -> Connector_PinSocket_1.27mm:PinSocket_2x03_P1.27mm_Vertical
Changed lines of the file:
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@@
 			)
 		)
-		(property "Footprint" "Connector_PinHeader_1.00mm:PinHeader_2x05_P1.00mm_Vertical_SMD"
+		(property "Footprint" "Connector_PinHeader_1.00mm:PinHeader_2x06_P1.00mm_Vertical"
 			(at 128.27 124.46 0)
 			(hide yes)
@@
 			)
 		)
-		(property "Footprint" "Connector_PinSocket_1.00mm:PinSocket_2x03_P1.00mm_Vertical_SMD"
+		(property "Footprint" "Connector_PinSocket_1.27mm:PinSocket_2x03_P1.27mm_Vertical"
 			(at 160.02 124.46 0)
 			(hide yes)
