File: PCB Test/_restore_backup_2026-08-21T21-40-26-668/PCB Test.kicad_pcb (KiCad board)
At the start: 2 copper layers, 51.6 x 67.2 mm, 50 parts, among them J1 Conn_02x02_Odd_Even, J2 Conn_02x05_Odd_Even, J3 Conn_02x02_Counter_Clockwise, J4 Conn_02x02_Counter_Clockwise, J5 Conn_02x02_Counter_Clockwise, J6 Conn_02x03_Odd_Even, Q2 NMOS, Q3 NMOS, SW1 SW_Push, SW2 SW_Push, SW3 SW_Push, U1 ATmega4808-A, U5 MCP1700x-330xxTO

Commit message: I am COOKING with the final edits
Parts:
- J1: value Conn_02x02_Odd_Even -> Conn_02x02_Counter_Clockwise; footprint Connector_PinHeader_2.54mm:PinHeader_2x02_P2.54mm_Vertical -> Connector:NS-Tech_Grove_1x04_P2mm_Vertical
- J3, J4, J5: value Conn_02x02_Counter_Clockwise -> Conn_02x02_Odd_Even; footprint Connector_PinHeader_2.54mm:PinHeader_2x02_P2.54mm_Vertical -> Connector_Harwin:Harwin_LTek-Male_2x02_P2.00mm_Vertical
- moved J2 204.8 mm to (1.79, 1.79)
- moved J6 16.2 mm to (192.0, 110.0), turned to 180 degrees
- moved R8 7.43 mm to (136.0, 99.0), turned to 0 degrees
- moved R14 6.25 mm to (136.2, 108.5), turned to 0 degrees
- moved J3 5.54 mm to (140.8, 99.0), turned to -90 degrees
- moved R16 5.15 mm to (136.0, 118.2), turned to 0 degrees
- moved J4 4.86 mm to (140.8, 108.5), turned to -90 degrees
- moved J5 4.71 mm to (140.8, 118.0), turned to -90 degrees
- moved J1 3.03 mm to (162.8, 141.0), turned to -90 degrees
Connections:
- J1 pad 2: +4.8V -> Net-(D1-A)
- J1 pad 3: Net-(D1-A) -> Net-(D2-A)
- J1 pad 4: Net-(D2-A) -> +4.8V
- J3 pad 2: GND -> +3.3V
- J3 pad 3: ADC Sensor 3 -> GND
- J3 pad 4: +3.3V -> ADC Sensor 3
- J4 pad 2: GND -> +3.3V
- J4 pad 3: ADC Sensor 2 -> GND
- J4 pad 4: +3.3V -> ADC Sensor 2
- J5 pad 2: GND -> +3.3V
- J5 pad 3: ADC Sensor 1 -> GND
- J5 pad 4: +3.3V -> ADC Sensor 1
Routing:
- net Motor 2: track 20.5 -> 64.6 mm, vias 2 -> 0
- net Motor 1: track 18.4 -> 60.3 mm, vias 2 -> 0
- net DTR: track 30.4 -> 14.3 mm, vias 2 -> 0
- net UPDI Data: track 19.9 -> 6.76 mm
- net USART RX: track 24.2 -> 12.8 mm
- net USART TX: track 23.5 -> 12.2 mm
- net +3.3V: track 109.9 -> 104.3 mm
- net +4.8V: track 98.6 -> 102.7 mm
- net ADC Sensor 3: track 27.9 -> 23.8 mm
- net ADC Sensor 2: track 16.7 -> 13.0 mm
- net GND: track 18.6 -> 22.0 mm
- net RESET: track 26.2 -> 23.7 mm
- net ADC Sensor 1: track 15.6 -> 13.1 mm
- net Net-(J5-Pin_1): track 3.17 -> 3.85 mm
- net Net-(Q3-G): track 11.8 -> 12.4 mm
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Other:
- board text removed: "Peter Ladur Line Following Robot"
