File: PCB Test/_restore_backup_2026-08-21T21-40-26-668/PCB Test.kicad_sch (KiCad schematic)
At the start: 50 parts, among them J1 Conn_02x02_Odd_Even, J2 Conn_02x05_Odd_Even, J3 Conn_02x02_Counter_Clockwise, J4 Conn_02x02_Counter_Clockwise, J5 Conn_02x02_Counter_Clockwise, J6 Conn_02x03_Odd_Even, Q2 NMOS, Q3 NMOS, SW1 SW_Push, SW2 SW_Push, SW3 SW_Push, U1 ATmega4808-A, U5 MCP1700x-330xxTO

Commit message: I am COOKING with the final edits
Parts:
- removed J1: Conn_02x02_Odd_Even, Connector_PinHeader_2.54mm:PinHeader_2x02_P2.54mm_Vertical, symbol Connector_Generic:Conn_02x02_Odd_Even
- removed J3, J4, J5: Conn_02x02_Counter_Clockwise, Connector_PinHeader_2.54mm:PinHeader_2x02_P2.54mm_Vertical, symbol Connector_Generic:Conn_02x02_Counter_Clockwise
- added J1: Conn_02x02_Counter_Clockwise, Connector:NS-Tech_Grove_1x04_P2mm_Vertical, symbol Connector_Generic:Conn_02x02_Counter_Clockwise
- added J3, J4, J5: Conn_02x02_Odd_Even, Connector_Harwin:Harwin_LTek-Male_2x02_P2.00mm_Vertical, symbol Connector_Generic:Conn_02x02_Odd_Even
Connections:
- net +3.3V: now also J3.2 (Pin_2), J4.2 (Pin_2), J5.2 (Pin_2)
- net +4.8V: now also J1.1 (Pin_1), J1.4 (Pin_4)
- net ADC Sensor 1: now also J5.4 (Pin_4)
- net ADC Sensor 2: now also J4.4 (Pin_4)
- net ADC Sensor 3: now also J3.4 (Pin_4)
- net GND: now also J3.3 (Pin_3), J4.3 (Pin_3), J5.3 (Pin_3)
- net at C5.2, D1.2 (A), Q2.1 (D): now also J1.2 (Pin_2)
- net at R14.2: now also J4.1 (Pin_1)
- net at R8.2: now also J3.1 (Pin_1)
- net at C6.2, D2.2 (A), Q3.1 (D): now also J1.3 (Pin_3)
- net at R16.2: now also J5.1 (Pin_1)
