File: PCB/_restore_backup_2026-08-22T13-01-56-422/PCB Test.kicad_pcb (KiCad board)
At the start: 2 copper layers, 51.6 x 67.2 mm, 49 parts, among them J1 Conn_02x02_Odd_Even, J2 Conn_02x05_Odd_Even, J3 Conn_02x02_Counter_Clockwise, J4 Conn_02x02_Counter_Clockwise, J5 Conn_02x02_Counter_Clockwise, J6 Conn_02x03_Odd_Even, Q2 NMOS, Q3 NMOS, U1 ATmega4808-A, U5 MCP1700x-330xxTO

Commit message: Rename PCB project to LFR_ATMega4808 and reorganize project files
Routing:
- net +3.3V: track 109.9 -> 120.2 mm, vias 5 -> 8
Changed lines of the file:
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@@
+	)
+	(segment
+		(start 145.5 128.25)
+		(end 145.5 122.5)
+		(width 0.5)
+		(layer "F.Cu")
+		(net "+3.3V")
 	)
 	(segment
@@
 		(end 175.396396 120.34)
 		(width 0.3)
+		(layer "F.Cu")
+		(net "+3.3V")
+	)
+	(segment
+		(start 145.5 122.5)
+		(end 144 121)
+		(width 0.5)
 		(layer "F.Cu")
 		(net "+3.3V")
@@
 	)
 	(via
+		(at 144 121)
+		(size 0.6)
+		(drill 0.3)
+		(layers "F.Cu" "B.Cu")
+		(net "+3.3V")
+	)
+	(via
+		(at 143.75 118.75)
+		(size 0.6)
+		(drill 0.3)
+		(layers "F.Cu" "B.Cu")
+		(net "+3.3V")
+	)
+	(via
 		(at 141 114.5)
 		(size 0.6)
@@
 	(via
 		(at 165.50962 118.05)
+		(size 0.6)
+		(drill 0.3)
+		(layers "F.Cu" "B.Cu")
+		(net "+3.3V")
+	)
+	(via
+		(at 143.75 118.75)
 		(size 0.6)
 		(drill 0.3)
@@
 	)
 	(segment
+		(start 144 121)
+		(end 144 119)
+		(width 0.5)
+		(layer "B.Cu")
+		(net "+3.3V")
+	)
+	(segment
 		(start 141 119.46)
 		(end 139.04 117.5)
 		(width 0.5)
 		(layer "B.Cu")
+		(net "+3.3V")
+	)
+	(segment
+		(start 144 119)
+		(end 143.75 118.75)
+		(width 0.5)
+		(layer "B.Cu")
