File: PCB/PCB Test.kicad_sch (KiCad schematic)
At the start: 49 parts, among them J1 Conn_02x02_Odd_Even, J2 Conn_02x05_Odd_Even, J3 Conn_02x02_Counter_Clockwise, J4 Conn_02x02_Counter_Clockwise, J5 Conn_02x02_Counter_Clockwise, J6 Conn_02x03_Odd_Even, Q2 NMOS, Q3 NMOS, U1 ATmega4808-A, U5 MCP1700x-330xxTO

Commit message: Final touches, v1 is ready
Other:
- moved on the sheet: D2
