File: PCB_V2/LFR_ATMega4808_V2.kicad_sch (KiCad schematic)
At the start: 74 parts, among them J1 Conn_02x02_Odd_Even, J10 Conn_01x03, J11 Conn_01x03, J2 Conn_02x05_Odd_Even, J5 Conn_01x03, J6 Conn_02x03_Odd_Even, J7 Conn_02x02_Odd_Even, J8 Conn_01x03, J9 Conn_01x03, Q1 PMOS_Si2333DDS, Q10 NMOS_BSR802NL6327HTSA1, Q11 NMOS_BSR802NL6327HTSA1, Q5 NMOS_BSR802NL6327HTSA1, Q6 NMOS_BSR802NL6327HTSA1, Q7 NMOS_BSR802NL6327HTSA1, Q8 NMOS_BSR802NL6327HTSA1, Q9 PMOS_Si2333DDS, U1 ATmega4808-A, U5 MCP1700x-330xxTO

Commit message: Redid the vias under the MCU
Parts:
- renumbered TP_3.3V to TP_3.3V1, TP_4.8V to TP_4.8V1
Changed lines of the file:
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@@
 		(in_pos_files yes)
 		(dnp no)
-		(property "Reference" "TP_4.8V"
+		(property "Reference" "TP_4.8V1"
 			(at 123.19 87.63 90)
 			(show_name no)
@@
 			(project "LFR_ATMega4808_V2"
 				(path "/7fcd8b9a-e9e6-4d51-9258-8399f733a0d2"
-					(reference "TP_4.8V")
+					(reference "TP_4.8V1")
 					(unit 1)
 				)
@@
 		(in_pos_files yes)
 		(dnp no)
-		(property "Reference" "TP_3.3V"
+		(property "Reference" "TP_3.3V1"
 			(at 121.285 61.595 90)
 			(show_name no)
@@
 			(project "LFR_ATMega4808_V2"
 				(path "/7fcd8b9a-e9e6-4d51-9258-8399f733a0d2"
-					(reference "TP_3.3V")
+					(reference "TP_3.3V1")
 					(unit 1)
 				)
